File: BreaV4.sch (EAGLE design)
At the start: 31 parts, among them J1 XF2L-0535-1, J2 XF2L-0535-1, Q3 ABM-16MHZ, SW1 ESE31L11T, SW2 EVQ11U09K, U1 TPS62200, X1 22-23-2021

Commit message: Schematics/Board file commit
Parts:
- added SW3: LS12T2-T, NewPart:LS12T2-T
Connections:
- net GND: now also SW3.S1
- net PWRSW: now also U2.PD6(AIN0); no longer U2.PD5(T1)
- net REST: now also U2.PD5(T1); no longer U2.PD6(AIN0)
- net RST: now also SW3.S2
Changed lines of the file:
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@@
 <part name="P+10" library="supply1" deviceset="VCC" device=""/>
 <part name="LED2" library="led" deviceset="LST-C19HE1WT" device=""/>
+<part name="SW3" library="NewPart" deviceset="LS12T2-T" device=""/>
 </parts>
 <sheets>
@@
 <instance part="P+10" gate="VCC" x="101.6" y="10.16"/>
 <instance part="LED2" gate="G$1" x="106.68" y="-15.24"/>
+<instance part="SW3" gate="G$1" x="20.32" y="88.9" rot="R270"/>
 </instances>
 <busses>
@@
 <pinref part="C3" gate="G$1" pin="1"/>
 <pinref part="GND5" gate="1" pin="GND"/>
-<wire x1="15.24" y1="81.28" x2="5.08" y2="81.28" width="0.1524" layer="91"/>
+<wire x1="15.24" y1="81.28" x2="10.16" y2="81.28" width="0.1524" layer="91"/>
+<pinref part="SW3" gate="G$1" pin="S1"/>
+<wire x1="10.16" y1="81.28" x2="5.08" y2="81.28" width="0.1524" layer="91"/>
+<wire x1="15.24" y1="88.9" x2="10.16" y2="88.9" width="0.1524" layer="91"/>
+<wire x1="10.16" y1="88.9" x2="10.16" y2="81.28" width="0.1524" layer="91"/>
+<junction x="10.16" y="81.28"/>
 </segment>
 <segment>
@@
 <segment>
 <pinref part="C3" gate="G$1" pin="2"/>
-<wire x1="22.86" y1="81.28" x2="38.1" y2="81.28" width="0.1524" layer="91"/>
+<wire x1="22.86" y1="81.28" x2="30.48" y2="81.28" width="0.1524" layer="91"/>
 <label x="35.56" y="81.28" size="1.778" layer="95" rot="R90" xref="yes"/>
 <pinref part="U2" gate="U$1" pin="PC6(/RESET)"/>
+<pinref part="SW3" gate="G$1" pin="S2"/>
+<wire x1="30.48" y1="81.28" x2="38.1" y2="81.28" width="0.1524" layer="91"/>
+<wire x1="25.4" y1="88.9" x2="30.48" y2="88.9" width="0.1524" layer="91"/>
+<wire x1="30.48" y1="88.9" x2="30.48" y2="81.28" width="0.1524" layer="91"/>
+<junction x="30.48" y="81.28"/>
 </segment>
 <segment>
@@
 </segment>
 <segment>
-<pinref part="U2" gate="U$1" pin="PD6(AIN0)"/>
-<wire x1="86.36" y1="43.18" x2="93.98" y2="43.18" width="0.1524" layer="91"/>
-<label x="93.98" y="43.18" size="1.778" layer="95"/>
+<pinref part="U2" gate="U$1" pin="PD5(T1)"/>
+<wire x1="86.36" y1="45.72" x2="93.98" y2="45.72" width="0.1524" layer="91"/>
+<label x="93.98" y="45.72" size="1.778" layer="95"/>
 </segment>
 </net>
@@
 </segment>
 <segment>
-<pinref part="U2" gate="U$1" pin="PD5(T1)"/>
-<wire x1="86.36" y1="45.72" x2="93.98" y2="45.72" width="0.1524" layer="91"/>
-<label x="93.98" y="45.72" size="1.778" layer="95"/>
-</segment>
-</net>
+<pinref part="U2" gate="U$1" pin="PD6(AIN0)"/>
+<wire x1="86.36" y1="43.18" x2="93.98" y2="43.18" width="0.1524" layer="91"/>
+<label x="93.98" y="43.18" size="1.778" layer="95"/>
+</segment>
+</net>
