File: Truss-Power-V4.brd (EAGLE design)
At the start: 40.3 x 20.3 mm, 41 parts, among them J1 XF2L-0625-1, U1 TPS61090, U2 MCP73831T-2ACI/OT, U3 MAX17044, U5 SN74LVC1G123, U6 INVERTER-GATE, U7 74LVC1G02SE, X1 CON-1PIN, X2 MicroB, X3 CON-1PINB, X4 CON-1PIN, X5 CON-1PIN, X6 CON-1PIN

Commit message: SIM800 added
Parts:
- removed C1: 10uF, adafruit:C0805K
- removed C2: 2.2uF, rcl:C0805K
- removed C4: 100uF, NewPart:7343-METRIC
- removed C6: 1000pF, rcl:C0402
- removed C7, C8: 0.1uF, rcl:C0603
- removed D1, D2: (no value), diode:SOD523
- removed L1: 2.5uH, NewPart:CDRH5D28
- removed LED1: (no value), led:CHIP-LED0603
- removed R1: 2.4M, adafruit:R0603
- removed R13: 1K, resistor:R0402
- removed R14: 10K, resistor:R0402
- removed R2: 390K, adafruit:R0603
- removed R3: 1.8M, adafruit:R0603
- removed R4: 200K, adafruit:R0603
- removed R5: 1M, adafruit:R0603
- removed U1: TPS61090, NewPart:TPS61090
- removed U5: SN74LVC1G123, NewPart:SSOP8
- removed U6: INVERTER-GATE, NewPart:SOC70-5@1
- removed U7: 74LVC1G02SE, NewPart:SOC70-5
- added ADC, PWM: (no value), adafruit:1X01-CLEANBIG
- added C9: 10uF, microbuilder:0805-NO
- added SW1: KMR2, microbuilder:BTN_KMR2_4.6X2.8
- added TP1: TPTP11R, testpad:TP11R
- added U4: SIM800H/L, microbuilder:SIM800L
- moved X6 14.0 mm to (5.35, 3.36)
- moved X5 7.88 mm to (13.2, 3.01)
Connections:
- removed net EN_SIG: U1.11
- removed net FB: R3.2, R4.1, U1.14
- removed net LBI: R1.1, R2.2, U1.9
- removed net LBO: R5.2, U1.12
- removed net N$10: C6.2, U5.6
- removed net N$11: U7.1
- removed net N$12: U7.2
- removed net N$4: LED1.C, R13.2
- removed net N$5: D2.A, U6.4
- removed net N$8: C6.1, R14.2, U5.7
- removed net N$9: D1.C, D2.C, U5.2
- removed net PWR_OR_R: U5.5
- removed net SW: L1.2, U1.3, U1.4
- removed net VCC: C2.1, C4.1, R10.2, R3.1, R5.1, R8.2, U1.1, U1.15, U1.16, X6.P$1
- new net 1.8V: U4.16
- new net 2.8V: TP1.TP, U4.18
- new net ADC: ADC.1, U4.50
- new net GSM_ANT: U4.40
- new net HP+: U4.17
- new net MIC1+: U4.52
- new net MIC2+: U4.9
- new net MIC2-: U4.10
- new net NETSTAT: U4.64
- new net PWM: PWM.1, U4.26
- new net PWRKEY: SW1.B, SW1.B', U4.48
- new net PWRSTAT: U4.4
- new net RESET: U4.49
- new net RI: U4.68
- new net SIMCLK: U4.55
- new net SIMDATA: U4.14
- new net SIMRST: U4.15
- new net SPEAKER1+: U4.53
- new net SPEAKER2+: U4.51
- new net SPEAKER2-: U4.11
- new net UART_RXD: U4.31
- new net UART_TXD: U4.32
- new net VRTC: C9.1, U4.56
- net DETSW_P: no longer U6.2
- net GND: now also C9.2, SW1.A, SW1.A', U4.12, U4.2, U4.35, U4.37, U4.38, U4.39, U4.41, U4.43, U4.44, U4.45, U4.57, U4.58, U4.6, U4.67, U4.71, U4.72, U4.73, U4.76, U4.77, U4.78, U4.79, U4.8, U4.80, U4.81, U4.82, U4.83, U4.84, U4.85, U4.86, U4.87, U4.88; no longer C1.2, C2.2, C4.2, C7.2, C8.2, R13.1, R2.1, R4.2, U1.13, U1.5, U1.6, U1.7, U1.EXP, U5.1, U5.4, U6.3, U7.3
- net LEDSOC: no longer LED1.A
- net PWRSW_P: no longer D1.A
- net VBAT: now also R10.2, R8.2, U4.1, U4.42, X6.P$1; no longer C1.1, C7.1, L1.1, R1.2, R14.1, U1.10, U1.8, U5.3, U5.8, U6.5
- net VBUS: now also U4.7
Routing:
- net LBO: track 18.0 -> 0.00 mm, vias 2 -> 0
- net EN_SIG: track 14.6 -> 0.00 mm, vias 1 -> 0
- net VBAT: track 15.9 -> 2.32 mm, vias 11 -> 6
- net FB: track 11.8 -> 0.00 mm, vias 2 -> 0
- net VCC: track 11.0 -> 0.00 mm
- net LBI: track 6.14 -> 0.00 mm
- net PWR_OR_R: track 5.28 -> 0.00 mm
- net N$9: track 5.21 -> 0.00 mm
- net N$8: track 3.60 -> 0.00 mm
- net N$5: track 3.56 -> 0.00 mm
- net N$10: track 2.19 -> 0.00 mm
- net GND: track 21.8 -> 19.8 mm, vias 8 -> 7
- net N$4: track 1.45 -> 0.00 mm
- net DETSW_P: track 4.67 -> 3.67 mm
- removed copper zone on layer 1, net SW
- removed copper zone on layer 1, net VCC

Commit message: Connectors updated
Parts:
- removed X1, X4, X5, X6: CON-1PIN, NewPart:CON-1PIN
- removed X3: CON-1PINB, NewPart:CON-1PIN-B
- added JP1, JP2: (no value), jumper:JP1
Connections:
- removed net DETSW_P: J1.4
- removed net LEDSOC: X3.P$1
- removed net PWRSW_P: J1.3
- removed net SHUTDOWN_SIG: J1.1
- net GND: now also JP2.1, JP2.2; no longer X1.P$1, X5.P$1
- net VBAT: now also JP1.1, JP1.2; no longer X4.P$1, X6.P$1
Routing:
- net LEDSOC: track 30.3 -> 0.00 mm
- net PWRSW_P: track 5.03 -> 0.00 mm
- net DETSW_P: track 3.67 -> 0.00 mm
- net SHUTDOWN_SIG: track 3.07 -> 0.00 mm
Changed lines of the file:
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@@
 <element name="C5" library="rcl" package="C0603" value="1uF" x="12.6238" y="14.5034"/>
 <element name="R7" library="resistor" package="R0402" value="470" x="38.92" y="14.52" rot="MR90"/>
-<element name="X4" library="NewPart" package="CON-1PIN" value="CON-1PIN" x="1.98" y="3.45" rot="R180"/>
-<element name="X5" library="NewPart" package="CON-1PIN" value="CON-1PIN" x="13.25" y="3.01" rot="R180"/>
 <element name="J1" library="con-omron" library_urn="urn:adsk.eagle:library:167" package="XF2L-0625-1" package3d_urn="urn:adsk.eagle:package:9011/1" value="XF2L-0625-1" x="4.68" y="8.26" rot="MR90">
 <attribute name="MF" value="OMRON COMPONENTS USA" x="4.68" y="8.26" size="1.778" layer="28" rot="MR90" display="off"/>
@@
 <attribute name="OC_NEWARK" value="29C7842" x="4.68" y="8.26" size="1.778" layer="28" rot="MR90" display="off"/>
 </element>
-<element name="X1" library="NewPart" package="CON-1PIN" value="CON-1PIN" x="15.95" y="2.88"/>
-<element name="X6" library="NewPart" package="CON-1PIN" value="CON-1PIN" x="5.35" y="3.36"/>
-<element name="X3" library="NewPart" package="CON-1PIN-B" value="CON-1PINB" x="7.26" y="15.61"/>
 <element name="U4" library="microbuilder" package="SIM800L" value="SIM800H/L" x="0.27" y="-25.78"/>
 <element name="SW1" library="microbuilder" package="BTN_KMR2_4.6X2.8" value="KMR2" x="10.41" y="-55.55"/>
@@
 <attribute name="TP_SIGNAL_NAME" value="" x="-13.21" y="-77.81" size="1.778" layer="27" display="off"/>
 </element>
+<element name="JP1" library="jumper" library_urn="urn:adsk.eagle:library:252" package="JP1" package3d_urn="urn:adsk.eagle:package:15455/1" value="" x="3.25" y="3.47" rot="R90"/>
+<element name="JP2" library="jumper" library_urn="urn:adsk.eagle:library:252" package="JP1" package3d_urn="urn:adsk.eagle:package:15455/1" value="" x="14.82" y="3.29" rot="R90"/>
 </elements>
 <signals>
@@
 <via x="13.7696" y="11.8738" extent="1-16" drill="0.5"/>
 <via x="7.9554" y="13.1226" extent="1-16" drill="0.5"/>
-<wire x1="23.78" y1="15.89" x2="23.78" y2="15.89" width="0" layer="19" extent="1-16"/>
 <via x="26.45" y="2.1" extent="1-16" drill="0.5"/>
 <via x="27.73" y="2.1" extent="1-16" drill="0.5"/>
@@
 <wire x1="37.8664" y1="9.4928" x2="36.954865625" y2="9.4928" width="0.8128" layer="1"/>
 <wire x1="36.954865625" y1="9.4928" x2="36.654865625" y2="9.1928" width="0.8128" layer="1"/>
-<contactref element="X5" pad="P$1"/>
-<contactref element="X1" pad="P$1"/>
 <contactref element="U4" pad="81"/>
 <contactref element="U4" pad="77"/>
@@
 <contactref element="U4" pad="57"/>
 <contactref element="U4" pad="12"/>
+<contactref element="JP2" pad="2"/>
+<contactref element="JP2" pad="1"/>
 <wire x1="12.46" y1="-54.75" x2="8.36" y2="-54.75" width="0" layer="19" extent="1-1"/>
 <wire x1="15.57" y1="-55.1" x2="12.46" y2="-54.75" width="0" layer="19" extent="1-1"/>
@@
 <wire x1="-7.83" y1="-29.98" x2="-4.63" y2="-32.88" width="0" layer="19" extent="1-1"/>
 <wire x1="-7.83" y1="-27.18" x2="-7.83" y2="-29.98" width="0" layer="19" extent="1-1"/>
-<wire x1="13.25" y1="3.01" x2="2.37" y2="-18.68" width="0" layer="19" extent="1-1"/>
+<wire x1="13.55" y1="3.29" x2="2.37" y2="-18.68" width="0" layer="19" extent="1-1"/>
 </signal>
 <signal name="N$14">
@@
 <via x="15.94" y="17.56" extent="1-16" drill="0.5"/>
 <contactref element="R6" pad="1"/>
-<contactref element="X4" pad="P$1"/>
 <contactref element="J1" pad="2"/>
 <via x="5.58" y="8.85" extent="1-16" drill="0.5"/>
-<wire x1="4.36" y1="15.29" x2="4.37" y2="15.28" width="0.254" layer="1"/>
 <wire x1="5.43" y1="10.165" x2="5.43" y2="9" width="0.254" layer="16"/>
 <wire x1="5.58" y1="8.85" x2="5.43" y2="9" width="0.254" layer="16"/>
@@
 <contactref element="R10" pad="2"/>
 <wire x1="12.4152" y1="7.1628" x2="12.4724" y2="7.22" width="0.254" layer="1"/>
-<contactref element="X6" pad="P$1"/>
+<contactref element="JP1" pad="2"/>
+<contactref element="JP1" pad="1"/>
 <wire x1="-7.43" y1="-18.68" x2="-7.83" y2="-20.18" width="0" layer="19" extent="1-1"/>
-<wire x1="1.98" y1="3.45" x2="-7.43" y2="-18.68" width="0" layer="19" extent="1-1"/>
+<wire x1="1.98" y1="3.47" x2="-7.43" y2="-18.68" width="0" layer="19" extent="1-1"/>
 <wire x1="10.466" y1="5.7102" x2="6.36" y2="8.99" width="0" layer="19" extent="1-16"/>
 <wire x1="12.4152" y1="7.1628" x2="10.466" y2="5.7102" width="0" layer="19" extent="1-1"/>
@@
 <wire x1="9.8188" y1="15.7184" x2="9.8386" y2="15.6986" width="0.254" layer="1"/>
 </signal>
-<signal name="LEDSOC">
-<wire x1="31.55" y1="19.83" x2="31.95" y2="19.43" width="0.254" layer="16"/>
-<wire x1="31.95" y1="19.43" x2="31.95" y2="17.18" width="0.254" layer="16"/>
-<contactref element="X3" pad="P$1"/>
-<wire x1="10.19" y1="19.83" x2="31.55" y2="19.83" width="0.254" layer="16"/>
-<wire x1="9.87" y1="19.51" x2="10.19" y2="19.83" width="0.254" layer="16"/>
-<wire x1="7.26" y1="15.61" x2="8.07" y2="16.42" width="0.254" layer="16"/>
-<wire x1="8.07" y1="16.42" x2="9.23" y2="16.42" width="0.254" layer="16"/>
-<wire x1="9.23" y1="16.42" x2="9.87" y2="17.06" width="0.254" layer="16"/>
-<wire x1="9.87" y1="17.06" x2="9.87" y2="19.51" width="0.254" layer="16"/>
-</signal>
-<signal name="PWRSW_P">
-<contactref element="J1" pad="3"/>
-<wire x1="4.93" y1="10.165" x2="4.93" y2="10.9" width="0.254" layer="16"/>
-<wire x1="4.93" y1="10.9" x2="2.98" y2="12.85" width="0.254" layer="16"/>
-<wire x1="2.98" y1="12.85" x2="2.98" y2="14.39" width="0.254" layer="16"/>
-</signal>
-<signal name="DETSW_P">
-<contactref element="J1" pad="4"/>
-<wire x1="4.17073125" y1="10.9444" x2="3.18926875" y2="10.9444" width="0.254" layer="16"/>
-<wire x1="3.18926875" y1="10.9444" x2="2.58486875" y2="10.34" width="0.254" layer="16"/>
-<wire x1="2.58486875" y1="10.34" x2="1.98" y2="10.34" width="0.254" layer="16"/>
-<wire x1="1.98" y1="10.34" x2="1.74" y2="10.58" width="0.254" layer="16"/>
-<wire x1="4.43" y1="10.165" x2="4.43" y2="10.68513125" width="0.254" layer="16"/>
-<wire x1="4.43" y1="10.68513125" x2="4.17073125" y2="10.9444" width="0.254" layer="16"/>
-</signal>
 <signal name="N$6">
 <contactref element="R7" pad="2"/>
@@
 <wire x1="35.3001" y1="16.9101" x2="35.72" y2="17.33" width="0.254" layer="1"/>
 </signal>
-<signal name="SHUTDOWN_SIG">
-<contactref element="J1" pad="1"/>
-<wire x1="5.93" y1="10.165" x2="5.93" y2="11.56" width="0.254" layer="16"/>
-<wire x1="5.93" y1="11.56" x2="5.2894" y2="12.2006" width="0.254" layer="16"/>
-<wire x1="5.2894" y1="12.49573125" x2="5.2894" y2="12.2006" width="0.254" layer="16"/>
-<wire x1="4.95513125" y1="12.83" x2="5.2894" y2="12.49573125" width="0.254" layer="16"/>
-</signal>
 <signal name="VRTC">
