File: Truss-Power-V4.sch (EAGLE design)
At the start: 41 parts, among them J1 XF2L-0625-1, U1 TPS61090, U2 MCP73831T-2ACI/OT, U3 MAX17044, U5 SN74LVC1G123, U6 INVERTER-GATE, U7 74LVC1G02SE, X1 CON-1PIN, X2 MicroB, X3 CON-1PINB, X4 CON-1PIN, X5 CON-1PIN, X6 CON-1PIN

Commit message: SIM800 added
Parts:
- removed C1: 10uF, adafruit:C-USC0805K
- removed C2: 2.2uF, rcl:C-EUC0805K
- removed C4: 100uF, NewPart:TANT-CAP
- removed C6: 1000pF, rcl:C-USC0402
- removed C7, C8: 0.1uF, rcl:C-USC0603
- removed D1, D2: (no value), diode:DIODE-SOD523
- removed L1: 2.5uH, NewPart:CDRH5D28
- removed LED1: (no value), led:LEDCHIP-LED0603
- removed R1: 2.4M, adafruit:R-US_R0603
- removed R13: 1K, resistor:R-US_R0402
- removed R14: 10K, resistor:R-US_R0402
- removed R2: 390K, adafruit:R-US_R0603
- removed R3: 1.8M, adafruit:R-US_R0603
- removed R4: 200K, adafruit:R-US_R0603
- removed R5: 1M, adafruit:R-US_R0603
- removed U1: TPS61090, NewPart:TPS61090
- removed U5: SN74LVC1G123, NewPart:SN74LVC1G123
- removed U6: INVERTER-GATE, NewPart:INVERTER-GATE
- removed U7: 74LVC1G02SE, NewPart:74LVC1G02SE
- added ADC, PWM: (no value), adafruit:PINHD-1X1CB
- added C9: 10uF, microbuilder:CAP_CERAMIC0805-NOOUTLINE
- added SW1: KMR2, microbuilder:SWITCH_TACT_SMT4.6X2.8
- added TP1: TPTP11R, testpad:TPTP11R
- added U4: SIM800H/L, microbuilder:GSM_SIM800L
Connections:
- removed net EN_SIG: U1.EN
- removed net FB: R3.2, R4.1, U1.FB
- removed net LBI: R1.1, R2.2, U1.LBI
- removed net LBO: R5.2, U1.LBO
- removed net N$10: C6.2, U5.C
- removed net N$11: U7.A
- removed net N$12: U7.B
- removed net N$4: LED1.C, R13.2
- removed net N$5: D2.A, U6.P$2
- removed net N$8: C6.1, R14.2, U5.R/C
- removed net N$9: D1.C, D2.C, U5.B
- removed net PWR_OR_R: U5.Q
- removed net SW: L1.2, U1.SW, U1.SW2
- removed net VCC: C2.1, C4.1, R10.2, R3.1, R5.1, R8.2, U1.VOUT, U1.VOUT2, U1.VOUT3, X6.P$1
- new net 1.8V: U4.VSIM
- new net 2.8V: TP1.TP, U4.VEXT
- new net ADC: ADC.1, U4.ADC
- new net GSM_ANT: U4.ANT
- new net HP+: U4.FM_ANT_P
- new net MIC1+: U4.MIC1P
- new net MIC2+: U4.MIC2P
- new net MIC2-: U4.MIC2N
- new net NETSTAT: U4.NETLIGHT
- new net PWM: PWM.1, U4.PWM
- new net PWRKEY: SW1.S, SW1.S1, U4.PWRKEY
- new net PWRSTAT: U4.STATUS
- new net RESET: U4.RESET
- new net RI: U4.UART_RI
- new net SIMCLK: U4.SIM_CLK
- new net SIMDATA: U4.SIM_DATA
- new net SIMRST: U4.SIM_RST
- new net SPEAKER1+: U4.SPK1P
- new net SPEAKER2+: U4.SPK2P/8Ω
- new net SPEAKER2-: U4.SPK2N
- new net UART_RXD: U4.UART_RXD
- new net UART_TXD: U4.UART_TXD
- new net VRTC: C9.1, U4.VRTC
- net DETSW_P: no longer U6.P$1
- net GND: now also C9.2, SW1.P, SW1.P1, U4.FM_ANT_N, U4.GND, U4.MIC1N; no longer C1.2, C2.2, C4.2, C7.2, C8.2, R13.1, R2.1, R4.2, U1.GND, U1.PAD, U1.PGND, U1.PGND2, U1.PGND3, U5./A, U5.GND, U6.GND, U7.GND
- net LEDSOC: no longer LED1.A
- net PWRSW_P: no longer D1.A
- net VBAT: now also R10.2, R8.2, U4.VBAT, X6.P$1; no longer C1.1, C7.1, L1.1, R1.2, R14.1, U1.SYNC, U1.VBAT, U5./CLR, U5.VCC, U6.VBAT
Other:
- note removed: "BOOST"
- note removed: "BOOST EN XOR"

Commit message: Connectors updated
Parts:
- removed X1, X4, X5, X6: CON-1PIN, NewPart:CON-1PIN
- removed X3: CON-1PINB, NewPart:CON-1PINB
- added JP1, JP2: (no value), jumper:JP1E
Connections:
- removed net DETSW_P: J1-4.MS
- removed net LEDSOC: X3.P$1
- removed net PWRSW_P: J1-3.MS
- removed net SHUTDOWN_SIG: J1-1.MS
- net GND: now also JP2.1, JP2.2; no longer X1.P$1, X5.P$1
- net VBAT: now also JP1.1, JP1.2; no longer X4.P$1, X6.P$1
Changed lines of the file:
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@@
 <part name="U$21" library="microbuilder" deviceset="VBAT" device=""/>
 <part name="R7" library="resistor" deviceset="R-US_" device="R0402" value="470"/>
-<part name="X4" library="NewPart" deviceset="CON-1PIN" device=""/>
-<part name="X5" library="NewPart" deviceset="CON-1PIN" device=""/>
 <part name="J1" library="con-omron" library_urn="urn:adsk.eagle:library:167" deviceset="XF2*-06?" device="25-1" package3d_urn="urn:adsk.eagle:package:9011/1" technology="L"/>
-<part name="X1" library="NewPart" deviceset="CON-1PIN" device=""/>
-<part name="X6" library="NewPart" deviceset="CON-1PIN" device=""/>
-<part name="X3" library="NewPart" deviceset="CON-1PINB" device=""/>
 <part name="U4" library="microbuilder" deviceset="GSM_SIM800L" device="" value="SIM800H/L"/>
 <part name="SW1" library="microbuilder" deviceset="SWITCH_TACT_SMT" device="4.6X2.8" value="KMR2"/>
@@
 <part name="TP1" library="testpad" deviceset="TP" device="TP11R"/>
 <part name="U$26" library="microbuilder" deviceset="GND" device=""/>
+<part name="JP1" library="jumper" library_urn="urn:adsk.eagle:library:252" deviceset="JP1E" device="" package3d_urn="urn:adsk.eagle:package:15455/1"/>
+<part name="JP2" library="jumper" library_urn="urn:adsk.eagle:library:252" deviceset="JP1E" device="" package3d_urn="urn:adsk.eagle:package:15455/1"/>
 </parts>
 <sheets>
@@
 </plain>
 <instances>
-<instance part="X4" gate="G$1" x="185.42" y="40.64"/>
-<instance part="X5" gate="G$1" x="185.42" y="35.56"/>
 <instance part="J1" gate="-1" x="127" y="60.96"/>
 <instance part="J1" gate="-2" x="127" y="58.42"/>
@@
 <instance part="J1" gate="-5" x="127" y="50.8"/>
 <instance part="J1" gate="-6" x="127" y="48.26"/>
-<instance part="X1" gate="G$1" x="185.42" y="55.88"/>
-<instance part="X6" gate="G$1" x="185.42" y="53.34"/>
-<instance part="X3" gate="G$1" x="127" y="38.1"/>
+<instance part="JP1" gate="A" x="170.18" y="45.72" rot="R90"/>
+<instance part="JP2" gate="A" x="170.18" y="38.1" rot="R90"/>
 </instances>
 <busses>
 </busses>
 <nets>
-<net name="GND" class="0">
-<segment>
-<pinref part="X5" gate="G$1" pin="P$1"/>
-<wire x1="180.34" y1="35.56" x2="175.26" y2="35.56" width="0.1524" layer="91"/>
-<label x="175.26" y="35.56" size="1.778" layer="95" rot="R180"/>
-</segment>
-<segment>
-<pinref part="X1" gate="G$1" pin="P$1"/>
-<wire x1="180.34" y1="55.88" x2="175.26" y2="55.88" width="0.1524" layer="91"/>
-<label x="175.26" y="55.88" size="1.778" layer="95" rot="R180"/>
-</segment>
-</net>
 <net name="VBAT" class="0">
 <segment>
@@
 </segment>
 <segment>
-<pinref part="X4" gate="G$1" pin="P$1"/>
-<wire x1="180.34" y1="40.64" x2="175.26" y2="40.64" width="0.1524" layer="91"/>
-<label x="175.26" y="40.64" size="1.778" layer="95" rot="R180"/>
-</segment>
-<segment>
-<pinref part="X6" gate="G$1" pin="P$1"/>
-<wire x1="180.34" y1="53.34" x2="175.26" y2="53.34" width="0.1524" layer="91"/>
-<label x="175.26" y="53.34" size="1.778" layer="95" rot="R180"/>
+<pinref part="JP1" gate="A" pin="2"/>
+<wire x1="172.72" y1="48.26" x2="180.34" y2="48.26" width="0.1524" layer="91"/>
+<label x="180.34" y="48.26" size="1.778" layer="95"/>
+</segment>
+<segment>
+<pinref part="JP1" gate="A" pin="1"/>
+<wire x1="172.72" y1="45.72" x2="180.34" y2="45.72" width="0.1524" layer="91"/>
+<label x="180.34" y="45.72" size="1.778" layer="95"/>
 </segment>
 </net>
@@
 </segment>
 </net>
-<net name="LEDSOC" class="0">
-<segment>
-<pinref part="X3" gate="G$1" pin="P$1"/>
-<wire x1="121.92" y1="38.1" x2="116.84" y2="38.1" width="0.1524" layer="91"/>
-<label x="116.84" y="38.1" size="1.778" layer="95" rot="R180"/>
-</segment>
-</net>
-<net name="PWRSW_P" class="0">
-<segment>
-<pinref part="J1" gate="-3" pin="MS"/>
-<wire x1="124.46" y1="55.88" x2="119.38" y2="55.88" width="0.1524" layer="91"/>
-<label x="114.3" y="55.88" size="1.778" layer="95"/>
-</segment>
-</net>
-<net name="DETSW_P" class="0">
-<segment>
-<pinref part="J1" gate="-4" pin="MS"/>
-<wire x1="124.46" y1="53.34" x2="119.38" y2="53.34" width="0.1524" layer="91"/>
-<label x="114.3" y="53.34" size="1.778" layer="95"/>
-</segment>
-</net>
-<net name="SHUTDOWN_SIG" class="0">
-<segment>
-<wire x1="124.46" y1="60.96" x2="119.38" y2="60.96" width="0.1524" layer="91"/>
-<label x="114.3" y="60.96" size="1.778" layer="95"/>
-<pinref part="J1" gate="-1" pin="MS"/>
-</segment>
-</net>
+<net name="GND" class="0">
+<segment>
+<pinref part="JP2" gate="A" pin="2"/>
+<wire x1="172.72" y1="40.64" x2="180.34" y2="40.64" width="0.1524" layer="91"/>
+<label x="180.34" y="40.64" size="1.778" layer="95"/>
+</segment>
+<segment>
+<pinref part="JP2" gate="A" pin="1"/>
+<wire x1="172.72" y1="38.1" x2="180.34" y2="38.1" width="0.1524" layer="91"/>
+<label x="180.34" y="38.1" size="1.778" layer="95"/>
+</segment>
+</net>
