File: TrussKeyV1/BreaV7.brd (EAGLE design)
At the start: 39.6 x 19 mm, 47 parts, among them J2 XF2L-0535-1, J3 XF2L-0635-1, Q1 ABM-16MHZ, SW1 LS12T2-T, SW2 EVQ11U09K, SW3 ESE31L11T, U2 TPS62200, U3 MCP73831T-2ACI/OT, U4 MAX17044, X1 CON-1PIN, X2 MicroB, X3 CON-1PIN

Commit message: 4-layer updated
Parts:
- removed C10, C12: 10µF, microbuilder:0805-NO
- removed C11: 10nF, rcl:C0603
- removed C13: 1uF, rcl:C0603
- removed CHRG: ORANGE, microbuilder:CHIPLED_0805_NOOUTLINE
- removed R10, R8: 4.7K, resistor:R0402
- removed R11: 1K, resistor:R0402
- removed R12: 180, resistor:R0402
- removed R13: 470, resistor:R0402
- removed R9: 2K, microbuilder:0805-NO
- removed U3: MCP73831T-2ACI/OT, microbuilder:SOT23-5
- removed U4: MAX17044, NewPart:TDFN
- removed X2: MicroB, microbuilder:4UCONN_20329
- added C14, C16: 10µF, microbuilder:0805-NO
- added C15: 10nF, rcl:C0603
- added C17: 1uF, rcl:C0603
- added CHRG1: ORANGE, microbuilder:CHIPLED_0805_NOOUTLINE
- added R14: 2K, microbuilder:0805-NO
- added R15, R16: 4.7K, resistor:R0402
- added R17: 1K, resistor:R0402
- added R18: 180, resistor:R0402
- added R19: 470, resistor:R0402
- added U5: MCP73831T-2ACI/OT, microbuilder:SOT23-5
- added U6: MAX17044, NewPart:TDFN
- added X4: MicroB, microbuilder:4UCONN_20329
- moved JP2 9.00 mm to (32.6, 16.2), turned to 0 degrees
- moved X3 2.85 mm to (37.0, 14.7)
Connections:
- removed net N$11: CHRG.C, U3.1
- removed net N$14: R9.1, U3.5
- removed net N$4: C13.1, R11.2, U4.2
- removed net N$6: C11.1, R12.2, U4.3
- removed net N$8: CHRG.A, R13.2
- removed net VBAT: C12.1, J2.1, J3.5, R10.2, R11.1, R12.1, R8.2, U3.3, X1.P$1
- removed net VBUS1: C10.1, R13.1, U3.4, X2.VBUS
- new net N$12: R14.1, U5.5
- new net N$13: C17.1, R17.2, U6.2
- new net N$15: C15.1, R18.2, U6.3
- new net N$16: CHRG1.A, R19.2
- new net N$17: CHRG1.C, U5.1
- new net VBUS2: C14.1, R19.1, U5.4, X4.VBUS
- net GND: now also C14.2, C15.2, C16.2, C17.2, R14.2, U5.2, U6.1, U6.4, U6.6, U6.9, X4.BASE@1, X4.BASE@2, X4.GND, X4.SPRT@1, X4.SPRT@2, X4.SPRT@3, X4.SPRT@4; no longer C10.2, C11.2, C12.2, C13.2, R9.2, U3.2, U4.1, U4.4, U4.6, U4.9, X2.BASE@1, X2.BASE@2, X2.GND, X2.SPRT@1, X2.SPRT@2, X2.SPRT@3, X2.SPRT@4
- net SCL: now also R16.1, U6.7; no longer R10.1, U4.7
- net SDA: now also R15.1, U6.8; no longer R8.1, U4.8
- net VCC: now also C16.1, J2.1, R15.2, R16.2, R17.1, R18.1, U5.3, X1.P$1
Routing:
- net VCC: track 87.6 -> 61.4 mm
- net VBAT: track 15.5 -> 0.00 mm
- net N$9: track 2.51 -> 6.72 mm
- added copper zone on layer 2, net GND
- added copper zone on layer 15, net VCC
