File: TrussKeyV1/BreaV7.sch (EAGLE design)
At the start: 47 parts, among them J2 XF2L-0535-1, J3 XF2L-0635-1, Q1 ABM-16MHZ, SW1 LS12T2-T, SW2 EVQ11U09K, SW3 ESE31L11T, U2 TPS62200, U3 MCP73831T-2ACI/OT, U4 MAX17044, X1 CON-1PIN, X2 MicroB, X3 CON-1PIN

Commit message: 4-layer updated
Parts:
- removed C10, C12: 10µF, microbuilder:CAP_CERAMIC0805-NOOUTLINE
- removed C11: 10nF, rcl:C-EUC0603
- removed C13: 1uF, rcl:C-EUC0603
- removed CHRG: ORANGE, microbuilder:LED0805_NOOUTLINE
- removed R10, R8: 4.7K, resistor:R-US_R0402
- removed R11: 1K, resistor:R-US_R0402
- removed R12: 180, resistor:R-US_R0402
- removed R13: 470, resistor:R-US_R0402
- removed R9: 2K, microbuilder:RESISTOR0805_NOOUTLINE
- removed U3: MCP73831T-2ACI/OT, microbuilder:MCP73831/2
- removed U4: MAX17044, NewPart:MAX17044
- removed X2: MicroB, microbuilder:USBMICRO_20329
- added C14, C16: 10µF, microbuilder:CAP_CERAMIC0805-NOOUTLINE
- added C15: 10nF, rcl:C-EUC0603
- added C17: 1uF, rcl:C-EUC0603
- added CHRG1: ORANGE, microbuilder:LED0805_NOOUTLINE
- added R14: 2K, microbuilder:RESISTOR0805_NOOUTLINE
- added R15, R16: 4.7K, resistor:R-US_R0402
- added R17: 1K, resistor:R-US_R0402
- added R18: 180, resistor:R-US_R0402
- added R19: 470, resistor:R-US_R0402
- added U5: MCP73831T-2ACI/OT, microbuilder:MCP73831/2
- added U6: MAX17044, NewPart:MAX17044
- added X4: MicroB, microbuilder:USBMICRO_20329
Connections:
- removed net N$11: CHRG.C, U3.STAT
- removed net N$14: R9.1, U3.PROG
- removed net N$4: C13.1, R11.2, U4.CELL
- removed net N$6: C11.1, R12.2, U4.VDD
- removed net N$8: CHRG.A, R13.2
- removed net VBAT: C12.1, J2-1.MSV, J3-5.MS, R10.2, R11.1, R12.1, R8.2, U3.VBAT, X1.P$1
- removed net VBUS1: C10.1, R13.1, U3.VDD, X2.VBUS
- new net N$12: R14.1, U5.PROG
- new net N$13: C17.1, R17.2, U6.CELL
- new net N$15: C15.1, R18.2, U6.VDD
- new net N$16: CHRG1.A, R19.2
- new net N$17: CHRG1.C, U5.STAT
- new net VBUS2: C14.1, R19.1, U5.VDD, X4.VBUS
- net GND: now also C14.2, C15.2, C16.2, C17.2, R14.2, U5.VSS, U6.CTG, U6.EPAD, U6.GND, U6.QSTRT, X4.GND; no longer C10.2, C11.2, C12.2, C13.2, R9.2, U3.VSS, U4.CTG, U4.EPAD, U4.GND, U4.QSTRT, X2.GND
- net SCL: now also R16.1, U6.SCL; no longer R10.1, U4.SCL
- net SDA: now also R15.1, U6.SDA; no longer R8.1, U4.SDA
- net VCC: now also C16.1, J2-1.MSV, R15.2, R16.2, R17.1, R18.1, U5.VBAT, X1.P$1
