File: TrussKeyV1/BreaV7.sch (EAGLE design)
At the start: 46 parts, among them J2 XF2L-0535-1, Q1 ABM-16MHZ, SW1 LS12T2-T, SW2 EVQ11U09K, SW3 ESE31L11T, U2 TPS62200, U5 MCP73831T-2ACI/OT, U6 MAX17044, X1 CON-1PIN, X3 CON-1PIN, X4 MicroB

Commit message: Layout
Parts:
- R19: value 470 -> 330
Changed lines of the file:
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@@
 <part name="U$25" library="microbuilder" deviceset="GND" device=""/>
 <part name="U$26" library="microbuilder" deviceset="VBAT" device=""/>
-<part name="R19" library="resistor" deviceset="R-US_" device="R0402" value="470"/>
+<part name="R19" library="resistor" deviceset="R-US_" device="R0402" value="330"/>
 <part name="R8" library="resistor" deviceset="R-US_" device="R0402" value="2K"/>
 </parts>

Commit message: V7 Gerber final
Changed lines of the file:
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@@
 <part name="U$11" library="microbuilder" deviceset="GND" device=""/>
 <part name="X4" library="microbuilder" deviceset="USB" device="MICRO_20329" value="MicroB"/>
-<part name="U$12" library="microbuilder" deviceset="VBAT" device=""/>
 <part name="P+12" library="supply1" deviceset="VCC" device=""/>
 <part name="R15" library="resistor" deviceset="R-US_" device="R0402" value="4.7K"/>
@@
 <instance part="U$11" gate="G$1" x="116.84" y="81.28"/>
 <instance part="X4" gate="G$1" x="25.4" y="104.14"/>
-<instance part="U$12" gate="G$1" x="134.62" y="116.84"/>
 <instance part="P+12" gate="VCC" x="86.36" y="60.96"/>
 <instance part="R15" gate="G$1" x="86.36" y="48.26" rot="R90"/>
@@
 <wire x1="127" y1="109.22" x2="101.6" y2="109.22" width="0.1524" layer="91"/>
 <wire x1="134.62" y1="109.22" x2="134.62" y2="114.3" width="0.1524" layer="91"/>
-<pinref part="U$12" gate="G$1" pin="VBAT"/>
 <pinref part="C16" gate="G$1" pin="1"/>
 <junction x="127" y="109.22"/>
-</segment>
-<segment>
+<label x="134.62" y="114.3" size="1.778" layer="95"/>
+</segment>
+<segment>

Commit message: Fusion PCBA
Parts:
- removed C15: 10nF, rcl:C-EUC0603
- removed R17: 1K, resistor:R-US_R0402
- removed R18: 180, resistor:R-US_R0402
- removed U6: MAX17044, NewPart:MAX17044
- added U3: LC709203, NewPart:LC709203
- R15, R16: value 4.7K -> 10K
- R7: value 330 -> 1K
Connections:
- removed net N$13: C17.1, R17.2, U6.CELL
- removed net N$15: C15.1, R18.2, U6.VDD
- new net VBAT: C17.2, U3.VDD
- net GND: now also C17.1, U3.EPAD, U3.TEST, U3.VSS; no longer C15.2, C17.2, U6.CTG, U6.EPAD, U6.GND, U6.QSTRT
- net SCL: now also R15.1, U3.SCL; no longer R16.1, U6.SCL
- net SDA: now also R16.1, U3.SDA; no longer R15.1, U6.SDA
- net VCC: no longer R17.1, R18.1
Other:
- moved on the sheet: C17
Changed lines of the file:
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@@
 <part name="C6" library="rcl" deviceset="C-EU" device="C0402" value="4.7uF"/>
 <part name="GND12" library="supply1" deviceset="GND" device=""/>
-<part name="R7" library="resistor" deviceset="R-US_" device="R0402" value="330"/>
+<part name="R7" library="resistor" deviceset="R-US_" device="R0402" value="1K"/>
 <part name="P+10" library="supply1" deviceset="VCC" device=""/>
 <part name="U1" library="SparkFun-DigitalIC" deviceset="ATMEGA328P_MLF" device="MLF32"/>
@@
 <part name="X4" library="microbuilder" deviceset="USB" device="MICRO_20329" value="MicroB"/>
 <part name="P+12" library="supply1" deviceset="VCC" device=""/>
-<part name="R15" library="resistor" deviceset="R-US_" device="R0402" value="4.7K"/>
-<part name="R16" library="resistor" deviceset="R-US_" device="R0402" value="4.7K"/>
-<part name="C15" library="rcl" deviceset="C-EU" device="C0603" value="10nF"/>
-<part name="U$13" library="microbuilder" deviceset="GND" device=""/>
+<part name="R15" library="resistor" deviceset="R-US_" device="R0402" value="10K"/>
+<part name="R16" library="resistor" deviceset="R-US_" device="R0402" value="10K"/>
 <part name="U$14" library="microbuilder" deviceset="GND" device=""/>
 <part name="U$16" library="microbuilder" deviceset="VBAT" device=""/>
 <part name="C16" library="microbuilder" deviceset="CAP_CERAMIC" device="0805-NOOUTLINE" value="10µF"/>
 <part name="U$17" library="microbuilder" deviceset="GND" device=""/>
-<part name="U6" library="NewPart" deviceset="MAX17044" device=""/>
-<part name="R17" library="resistor" deviceset="R-US_" device="R0402" value="1K"/>
-<part name="R18" library="resistor" deviceset="R-US_" device="R0402" value="180"/>
-<part name="U$22" library="microbuilder" deviceset="GND" device=""/>
 <part name="U$23" library="microbuilder" deviceset="GND" device=""/>
-<part name="U$24" library="microbuilder" deviceset="GND" device=""/>
 <part name="C17" library="rcl" deviceset="C-EU" device="C0603" value="1uF"/>
-<part name="U$25" library="microbuilder" deviceset="GND" device=""/>
-<part name="U$26" library="microbuilder" deviceset="VBAT" device=""/>
 <part name="R19" library="resistor" deviceset="R-US_" device="R0402" value="330"/>
 <part name="R8" library="resistor" deviceset="R-US_" device="R0402" value="2K"/>
+<part name="U3" library="NewPart" deviceset="LC709203" device=""/>
+<part name="U$1" library="microbuilder" deviceset="GND" device=""/>
 </parts>
 <sheets>
@@
 <instance part="R15" gate="G$1" x="86.36" y="48.26" rot="R90"/>
 <instance part="R16" gate="G$1" x="104.14" y="43.18" rot="R90"/>
-<instance part="C15" gate="G$1" x="40.64" y="17.78"/>
-<instance part="U$13" gate="G$1" x="48.26" y="7.62"/>
 <instance part="U$14" gate="G$1" x="93.98" y="25.4"/>
-<instance part="U$16" gate="G$1" x="20.32" y="22.86"/>
+<instance part="U$16" gate="G$1" x="25.4" y="25.4"/>
 <instance part="C16" gate="G$1" x="127" y="104.14"/>
 <instance part="U$17" gate="G$1" x="127" y="96.52"/>
-<instance part="U6" gate="G$1" x="66.04" y="27.94"/>
-<instance part="R17" gate="G$1" x="33.02" y="33.02"/>
-<instance part="R18" gate="G$1" x="33.02" y="20.32"/>
-<instance part="U$22" gate="G$1" x="40.64" y="7.62"/>
 <instance part="U$23" gate="G$1" x="43.18" y="35.56"/>
-<instance part="U$24" gate="G$1" x="93.98" y="20.32"/>
-<instance part="C17" gate="G$1" x="45.72" y="30.48"/>
-<instance part="U$25" gate="G$1" x="40.64" y="22.86"/>
-<instance part="U$26" gate="G$1" x="20.32" y="35.56"/>
+<instance part="C17" gate="G$1" x="40.64" y="30.48"/>
 <instance part="R19" gate="G$1" x="57.15" y="104.14" rot="MR180"/>
 <instance part="R8" gate="G$1" x="110.49" y="106.68" rot="MR180"/>
+<instance part="U3" gate="U1" x="63.5" y="27.94"/>
+<instance part="U$1" gate="G$1" x="30.48" y="30.48"/>
 </instances>
 <busses>
@@
 <pinref part="U$14" gate="G$1" pin="GND"/>
 <wire x1="78.74" y1="27.94" x2="93.98" y2="27.94" width="0.1524" layer="91"/>
-<pinref part="U6" gate="G$1" pin="EPAD"/>
+<pinref part="U3" gate="U1" pin="EPAD"/>
 </segment>
 <segment>
@@
 </segment>
 <segment>
-<wire x1="48.26" y1="17.78" x2="48.26" y2="10.16" width="0.1524" layer="91"/>
-<pinref part="U6" gate="G$1" pin="GND"/>
-<pinref part="U$13" gate="G$1" pin="GND"/>
-</segment>
-<segment>
-<pinref part="C15" gate="G$1" pin="2"/>
-<pinref part="U$22" gate="G$1" pin="GND"/>
-<wire x1="40.64" y1="12.7" x2="40.64" y2="10.16" width="0.1524" layer="91"/>
-</segment>
-<segment>
 <pinref part="U$23" gate="G$1" pin="GND"/>
-<pinref part="U6" gate="G$1" pin="CTG"/>
 <wire x1="43.18" y1="38.1" x2="48.26" y2="38.1" width="0.1524" layer="91"/>
-</segment>
-<segment>
-<pinref part="U6" gate="G$1" pin="QSTRT"/>
-<pinref part="U$24" gate="G$1" pin="GND"/>
-<wire x1="78.74" y1="22.86" x2="93.98" y2="22.86" width="0.1524" layer="91"/>
-</segment>
-<segment>
-<pinref part="C17" gate="G$1" pin="2"/>
-<pinref part="U$25" gate="G$1" pin="GND"/>
-<wire x1="45.72" y1="25.4" x2="40.64" y2="25.4" width="0.1524" layer="91"/>
+<pinref part="U3" gate="U1" pin="TEST"/>
+</segment>
+<segment>
+<pinref part="U3" gate="U1" pin="VSS"/>
+<pinref part="C17" gate="G$1" pin="1"/>
+<wire x1="48.26" y1="33.02" x2="40.64" y2="33.02" width="0.1524" layer="91"/>
+<pinref part="U$1" gate="G$1" pin="GND"/>
+<wire x1="40.64" y1="33.02" x2="30.48" y2="33.02" width="0.1524" layer="91"/>
+<junction x="40.64" y="33.02"/>
 </segment>
 </net>
@@
 <junction x="127" y="109.22"/>
 <label x="134.62" y="114.3" size="1.778" layer="95"/>
-</segment>
-<segment>
-<pinref part="U$16" gate="G$1" pin="VBAT"/>
-<pinref part="R18" gate="G$1" pin="1"/>
-<wire x1="20.32" y1="20.32" x2="27.94" y2="20.32" width="0.1524" layer="91"/>
-</segment>
-<segment>
-<pinref part="U$26" gate="G$1" pin="VBAT"/>
-<pinref part="R17" gate="G$1" pin="1"/>
-<wire x1="20.32" y1="33.02" x2="27.94" y2="33.02" width="0.1524" layer="91"/>
 </segment>
 <segment>
@@
 <wire x1="104.14" y1="55.88" x2="86.36" y2="55.88" width="0.1524" layer="91"/>
 <junction x="86.36" y="55.88"/>
-</segment>
-</net>
-<net name="SCL" class="0">
-<segment>
-<wire x1="99.06" y1="33.02" x2="104.14" y2="33.02" width="0.1524" layer="91"/>
-<label x="109.22" y="33.02" size="1.778" layer="95" xref="yes"/>
-<pinref part="R16" gate="G$1" pin="1"/>
-<wire x1="104.14" y1="33.02" x2="109.22" y2="33.02" width="0.1524" layer="91"/>
-<wire x1="78.74" y1="33.02" x2="104.14" y2="33.02" width="0.1524" layer="91"/>
-<wire x1="104.14" y1="33.02" x2="104.14" y2="38.1" width="0.1524" layer="91"/>
-<junction x="104.14" y="33.02"/>
-<pinref part="U6" gate="G$1" pin="SCL"/>
-</segment>
-</net>
-<net name="SDA" class="0">
-<segment>
-<wire x1="86.36" y1="38.1" x2="91.44" y2="38.1" width="0.1524" layer="91"/>
-<label x="91.44" y="38.1" size="1.778" layer="95" xref="yes"/>
-<pinref part="R15" gate="G$1" pin="1"/>
-<wire x1="78.74" y1="38.1" x2="86.36" y2="38.1" width="0.1524" layer="91"/>
-<wire x1="86.36" y1="38.1" x2="86.36" y2="43.18" width="0.1524" layer="91"/>
-<junction x="86.36" y="38.1"/>
-<pinref part="U6" gate="G$1" pin="SDA"/>
 </segment>
 </net>
@@
 </segment>
 </net>
-<net name="N$13" class="0">
-<segment>
-<pinref part="U6" gate="G$1" pin="CELL"/>
-<pinref part="C17" gate="G$1" pin="1"/>
-<wire x1="45.72" y1="33.02" x2="48.26" y2="33.02" width="0.1524" layer="91"/>
-<pinref part="R17" gate="G$1" pin="2"/>
-<wire x1="38.1" y1="33.02" x2="45.72" y2="33.02" width="0.1524" layer="91"/>
-</segment>
-</net>
-<net name="N$15" class="0">
-<segment>
-<pinref part="C15" gate="G$1" pin="1"/>
-<pinref part="R18" gate="G$1" pin="2"/>
-<wire x1="38.1" y1="20.32" x2="40.64" y2="20.32" width="0.1524" layer="91"/>
-<pinref part="U6" gate="G$1" pin="VDD"/>
-<wire x1="40.64" y1="20.32" x2="48.26" y2="20.32" width="0.1524" layer="91"/>
-<wire x1="48.26" y1="20.32" x2="48.26" y2="22.86" width="0.1524" layer="91"/>
-</segment>
-</net>
 <net name="N$16" class="0">
 <segment>
@@
 </segment>
 </net>
+<net name="SCL" class="0">
+<segment>
+<pinref part="U3" gate="U1" pin="SCL"/>
+<pinref part="R15" gate="G$1" pin="1"/>
+<wire x1="78.74" y1="38.1" x2="86.36" y2="38.1" width="0.1524" layer="91"/>
+<wire x1="86.36" y1="38.1" x2="86.36" y2="43.18" width="0.1524" layer="91"/>
+<label x="86.36" y="38.1" size="1.778" layer="95"/>
+</segment>
+</net>
+<net name="SDA" class="0">
+<segment>
+<pinref part="U3" gate="U1" pin="SDA"/>
+<pinref part="R16" gate="G$1" pin="1"/>
+<wire x1="78.74" y1="33.02" x2="104.14" y2="33.02" width="0.1524" layer="91"/>
+<wire x1="104.14" y1="33.02" x2="104.14" y2="38.1" width="0.1524" layer="91"/>
+<label x="104.14" y="33.02" size="1.778" layer="95"/>
+</segment>
+</net>
+<net name="VBAT" class="0">
+<segment>
+<pinref part="U3" gate="U1" pin="VDD"/>
+<wire x1="48.26" y1="22.86" x2="40.64" y2="22.86" width="0.1524" layer="91"/>
+<pinref part="U$16" gate="G$1" pin="VBAT"/>
+<wire x1="40.64" y1="22.86" x2="25.4" y2="22.86" width="0.1524" layer="91"/>
+<pinref part="C17" gate="G$1" pin="2"/>
+<wire x1="40.64" y1="25.4" x2="40.64" y2="22.86" width="0.1524" layer="91"/>
+<junction x="40.64" y="22.86"/>
+</segment>
+</net>
